File: SlimeDongle-ESP.kicad_pcb (KiCad board)
At the start: 2 copper layers, 18.1 x 39.4 mm, 20 parts, among them J1 USB_A, SW1 FLASH, U1 M3406, U3 ESP-12F

Commit message: added jlc pcba tooling holes
Parts:
- added REF**: ToolingHoleJLC, SlimeDongle-ESP_Footprints:ToolingHoleJLC, F.Cu at (134.4, 112.0)
- added REF**: ToolingHoleJLC, SlimeDongle-ESP_Footprints:ToolingHoleJLC, F.Cu at (150.0, 112.0)
- added REF**: ToolingHoleJLC, SlimeDongle-ESP_Footprints:ToolingHoleJLC, F.Cu at (146.0, 74.8)
Changed lines of the file:
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@@
     )
+  )
+  (footprint "SlimeDongle-ESP_Footprints:ToolingHoleJLC" (layer "F.Cu")
+    (at 134.4 112)
+    (attr through_hole)
+    (fp_text reference "REF**" (at 0 -0.5 unlocked) (layer "F.SilkS") hide
+        (effects (font (size 1 1) (thickness 0.1)))
+    )
+    (fp_text value "ToolingHoleJLC" (at 0 1 unlocked) (layer "F.Fab") hide
+        (effects (font (size 1 1) (thickness 0.15)))
+    )
+    (pad "" np_thru_hole circle (at 0 0) (size 1.152 1.152) (drill 1.152) (layers "F&B.Cu" "*.Mask")
+      (solder_mask_margin 0.148) (clearance 0.248) (zone_connect 0))
   )
   (footprint "SlimeDongle-ESP_Footprints:C_0603_1608Metric_Pad1.08x0.95mm_HandSolder" (layer "F.Cu")
@@
       (rotate (xyz -90 0 -90))
     )
+  )
+  (footprint "SlimeDongle-ESP_Footprints:ToolingHoleJLC" (layer "F.Cu")
+    (at 150 112)
+    (attr through_hole)
+    (fp_text reference "REF**" (at 0 -0.5 unlocked) (layer "F.SilkS") hide
+        (effects (font (size 1 1) (thickness 0.1)))
+    )
+    (fp_text value "ToolingHoleJLC" (at 0 1 unlocked) (layer "F.Fab") hide
+        (effects (font (size 1 1) (thickness 0.15)))
+    )
+    (pad "" np_thru_hole circle (at 0 0) (size 1.152 1.152) (drill 1.152) (layers "F&B.Cu" "*.Mask")
+      (solder_mask_margin 0.148) (clearance 0.248) (zone_connect 0))
   )
   (footprint "SlimeDongle-ESP_Footprints:C_0603_1608Metric_Pad1.08x0.95mm_HandSolder" (layer "F.Cu")
@@
     )
   )
+  (footprint "SlimeDongle-ESP_Footprints:ToolingHoleJLC" (layer "F.Cu")
+    (at 146 74.8)
+    (attr through_hole)
+    (fp_text reference "REF**" (at 0 -0.5 unlocked) (layer "F.SilkS") hide
+        (effects (font (size 1 1) (thickness 0.1)))
+    )
+    (fp_text value "ToolingHoleJLC" (at 0 1 unlocked) (layer "F.Fab") hide
+        (effects (font (size 1 1) (thickness 0.15)))
+    )
+    (pad "" np_thru_hole circle (at 0 0) (size 1.152 1.152) (drill 1.152) (layers "F&B.Cu" "*.Mask")
+      (solder_mask_margin 0.148) (clearance 0.248) (zone_connect 0))
+  )
   (footprint "SlimeDongle-ESP_Footprints:SOT-23-5" (layer "F.Cu")

Commit message: 1.1
Parts:
- removed the G*** at (142.4, 82.4)
- removed the REF** at (134.4, 112.0)
- removed the REF** at (150.0, 112.0)
- removed the REF** at (146.0, 74.8)
- added G***: LOGO, SlimeDongle-ESP_Footprints:Luna5x5, F.Cu at (115.1, 129.8)
- added REF**: ToolingHoleJLC, SlimeDongle-ESP_Footprints:ToolingHoleJLC, F.Cu at (109.5, 108.0)
- added REF**: ToolingHoleJLC, SlimeDongle-ESP_Footprints:ToolingHoleJLC, F.Cu at (101.5, 133.2)
- added REF**: ToolingHoleJLC, SlimeDongle-ESP_Footprints:ToolingHoleJLC, F.Cu at (117.5, 133.0)
- C1, C2, C3, C4, C5: footprint SlimeDongle-ESP_Footprints:C_0603_1608Metric_Pad1.08x0.95mm_HandSolder -> Capacitor_SMD:C_0603_1608Metric_Pad1.08x0.95mm_HandSolder
- D1: footprint SlimeDongle-ESP_Footprints:LED_0603_1608Metric_Pad1.05x0.95mm_HandSolder -> LED_SMD:LED_0603_1608Metric_Pad1.05x0.95mm_HandSolder
- J1: footprint SlimeDongle-ESP_Footprints:USB_A_CNCTech_1001-011-01101_Horizontal -> Connector_USB:USB_A_CNCTech_1001-011-01101_Horizontal
- L1: footprint SlimeDongle-ESP_Footprints:L_0603_1608Metric_Pad1.05x0.95mm_HandSolder -> Inductor_SMD:L_0603_1608Metric_Pad1.05x0.95mm_HandSolder
- R1, R2, R3, R4, R5, R6, R7: footprint SlimeDongle-ESP_Footprints:R_0603_1608Metric_Pad0.98x0.95mm_HandSolder -> Resistor_SMD:R_0603_1608Metric_Pad0.98x0.95mm_HandSolder
- SW1: footprint SlimeDongle-ESP_Footprints:SW_SPST_B3U-1000P -> Button_Switch_SMD:SW_SPST_B3U-1000P
- U1: footprint SlimeDongle-ESP_Footprints:SOT-23-5 -> Package_TO_SOT_SMD:SOT-23-5
- U2: footprint SlimeDongle-ESP_Footprints:SOP-8_3.9x4.9mm_P1.27mm -> Package_SO:SOP-8_3.9x4.9mm_P1.27mm
- U3: footprint SlimeDongle-ESP_Footprints:ESP-12E -> RF_Module:ESP-12E
- moved R2 46.5 mm to (110.8, 129.5), turned to 90 degrees
- moved U1 44.7 mm to (108.0, 126.9), turned to -90 degrees
- moved C1 44.7 mm to (108.0, 130.4), turned to 0 degrees
- moved C2 43.7 mm to (102.1, 123.1), turned to 0 degrees
- moved R3 43.7 mm to (105.8, 119.2), turned to 0 degrees
- moved U2 43.5 mm to (103.1, 127.9)
- moved R1 43.2 mm to (110.8, 125.9), turned to -90 degrees
- moved L1 43.1 mm to (105.8, 123.1)
- moved D1 43.1 mm to (109.5, 121.2)
- moved SW1 43.1 mm to (115.1, 122.8)
- moved J1 42.2 mm to (109.5, 143.8)
- moved C4 42.2 mm to (102.1, 119.2), turned to 0 degrees
- moved C5 42.2 mm to (102.1, 121.2), turned to 0 degrees
- moved R4 42.0 mm to (105.8, 121.2), turned to 0 degrees
- moved U3 42.0 mm to (109.5, 104.8)
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Routing:
- net +3V3: track 30.1 -> 21.9 mm, vias 5 -> 7
- net UART_TX: track 33.5 -> 40.0 mm
- net Net-(U3-GPIO12): track 10.3 -> 15.2 mm, vias 0 -> 2
- net Net-(U2-VCC): track 6.67 -> 3.71 mm
- net UART_RX: track 37.0 -> 39.8 mm
- net Net-(U3-EN): track 20.4 -> 17.8 mm
- net GND: track 6.42 -> 8.77 mm, vias 2 -> 3
- net Net-(U1-SW): track 1.96 -> 4.24 mm
- net Net-(SW1-A): track 14.8 -> 16.8 mm
- net D-: track 10.8 -> 12.6 mm
- net D+: track 9.92 -> 11.5 mm
- net Net-(U3-~{RST}): track 25.6 -> 25.8 mm, vias 2 -> 0
- net +5V: track 15.0 -> 15.1 mm, vias 2 -> 0
Other:
- board size 18.1 x 39.4 mm -> 19 x 40 mm
- board text removed: "SlimeDongle ESP8266"
- board text removed: "by Higanbana"
- board text removed: "v1.0"
